File: kicad/DCDCv9-3.kicad_sch (KiCad schematic)
At the start: 187 parts, among them J1 Screw_Terminal_01x03, J1.1 Screw_Terminal_01x03, J1.2 Screw_Terminal_01x03, J2 Conn_01x02_Male, J3 Conn_01x02, J3.1 Conn_01x02, J3.2 Conn_01x01_Pin, J3.3 Conn_01x01_Pin, J4 Conn_01x02_Male, J5 XT60 Male, J5.1 XT60 Female (wrong symbol ik), J6 Conn_01x02_Male, J7 Conn_01x02_Male, J8 Conn_01x02_Male, M1 Fan, Q1 PMV20ENR, Q10 IMBG65R050M2HXTMA1, Q11 IMBG65R050M2HXTMA1, Q2 PMV20ENR, Q3 SIHP24N80AE-GE3, Q4 IXYP8N90C3, Q5 PMV20ENR, Q6 PMV20ENR, Q7 PMV20ENR, T1 DIY Transformer ETD 39, T1.1 Ferrite Core, T1.2 Ferrite Core (gapped), T1.3 1800 mm 120 x 0.1 mm HF litz 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, T1.4 165 mm 600 x 0,071 mm HF litz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, T1.5 165 mm 600 x 0,071 mm HF litz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, U1 TBA 1-1212HI, U10 LM2904BIDDFR, U11 UCC21520DW, U12 UCC25600, U13 ZXRE330ASA-7, U14 LM2904BIDDFR, U2 RT9058-90GVL, U3 MP4541_SOP8-EP, U4 TLV61048DBVR, U6 LM2904BIDDFR, U7 TL431, U9 ACPL-217-50AE

Commit message: improved clearance on R54
Other:
- title: DC/DC v9-3 -> DC/DC v9-3.1
Changed lines of the file:
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@@
 	(paper "A3")
 	(title_block
-		(title "DC/DC v9-3")
-		(date "2025-01-26")
+		(title "DC/DC v9-3.1")
+		(date "2025-02-04")
 		(company "Author: Rootthecause")
 	)

Commit message: increased clearance a bit more
Other:
- title: DC/DC v9-3.1 -> DC/DC v9-3r1
Changed lines of the file:
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@@
 	(paper "A3")
 	(title_block
-		(title "DC/DC v9-3.1")
+		(title "DC/DC v9-3r1")
 		(date "2025-02-04")
 		(company "Author: Rootthecause")

Commit message: included LTspice simulation for precharge
Parts:
- U1: comment (none) -> If not available, use PD01S1212A https://www.mouser.de/Prod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
Changed lines of the file:
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@@
 			)
 		)
-		(property "comment" ""
+		(property "comment" "If not available, use PD01S1212A https://www.mouser.de/ProductDetail/Delta-Electronics/PD01S1212A?qs=%2FW4LtXOBxKsNNDIpmtt%2FbQ%3D%3D "
 			(at 50.8 53.34 0)
 			(effects

Commit message: fixed mixed up U_on/off comment at U6B, added PDF plot of schematic, replaced TL431 ED back to TL431
Other:
- note added: "R54 = 470k U_on = 5.9466 V = 4784.4 Ω = 1.2267 = 77 °C U_off = 6.0533 V = 4617.2 Ω = 1.1839 = 68 °C 106.7 mV hysteresis"
- note removed: "R54 = 470k U_on = 6.0533 V = 4617.2 Ω = 1.1839 = 68 °C U_off = 5.9466 V = 4784.4 Ω = 1.2267 = 77 °C 106.7 mV hysteresis"
Changed lines of the file:
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@@
 		)
 	)
-	(text "R54 = 470k\nU_on = 6.0533 V = 4617.2 Ω = 1.1839 = 68 °C\nU_off = 5.9466 V = 4784.4 Ω = 1.2267 = 77 °C\n106.7 mV hysteresis"
+	(text "R54 = 470k\nU_on = 5.9466 V = 4784.4 Ω = 1.2267 = 77 °C\nU_off = 6.0533 V = 4617.2 Ω = 1.1839 = 68 °C\n106.7 mV hysteresis"
 		(exclude_from_sim no)
 		(at 112.395 271.78 0)
